File: prototypes/motherboard-stage1/cpu_men.kicad_sch (KiCad schematic)
At the start: 15 parts, among them U1 MC6309, U2 28C64, U3 AS6C4008, Y2 12Mhz

Commit message: in between commits
Connections:
- net GND: no longer R6.1
- net MRDY: now also R6.1; no longer R6.2
- net VCC: now also R6.2
Other:
- moved on the sheet: R6
Changed lines of the file:
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@@
 	)
 	(junction
+		(at 63.5 113.03)
+		(diameter 0)
+		(color 0 0 0 0)
+	)
+	(junction
 		(at 55.88 105.41)
 		(diameter 0)
@@
 	)
 	(junction
-		(at 64.77 113.03)
+		(at 236.22 30.48)
 		(diameter 0)
 		(color 0 0 0 0)
 	)
 	(junction
-		(at 236.22 30.48)
+		(at 60.96 67.31)
 		(diameter 0)
 		(color 0 0 0 0)
@@
 		)
 	)
-	(wire
-		(pts
-			(xy 64.77 113.03) (xy 86.36 113.03)
-		)
-		(stroke
-			(width 0)
-			(type default)
-		)
-	)
 	(bus
 		(pts
@@
 	(wire
 		(pts
-			(xy 64.77 123.19) (xy 64.77 124.46)
-		)
-		(stroke
-			(width 0)
-			(type default)
-		)
-	)
-	(wire
-		(pts
 			(xy 222.25 80.01) (xy 233.68 80.01)
 		)
@@
 	(wire
 		(pts
-			(xy 59.69 113.03) (xy 64.77 113.03)
+			(xy 59.69 113.03) (xy 63.5 113.03)
 		)
 		(stroke
@@
 	(wire
 		(pts
+			(xy 63.5 76.2) (xy 63.5 113.03)
+		)
+		(stroke
+			(width 0)
+			(type default)
+		)
+	)
+	(wire
+		(pts
 			(xy 209.55 129.54) (xy 209.55 130.81)
 		)
@@
 		)
 	)
-	(wire
+	(bus
 		(pts
-			(xy 64.77 113.03) (xy 64.77 115.57)
+			(xy 184.15 105.41) (xy 184.15 107.95)
 		)
 		(stroke
@@
 		)
 	)
-	(bus
+	(wire
 		(pts
-			(xy 184.15 105.41) (xy 184.15 107.95)
+			(xy 63.5 68.58) (xy 63.5 67.31)
 		)
 		(stroke
@@
 	(wire
 		(pts
+			(xy 60.96 67.31) (xy 63.5 67.31)
+		)
+		(stroke
+			(width 0)
+			(type default)
+		)
+	)
+	(wire
+		(pts
 			(xy 135.89 90.17) (xy 146.05 90.17)
 		)
@@
 	(wire
 		(pts
+			(xy 63.5 113.03) (xy 86.36 113.03)
+		)
+		(stroke
+			(width 0)
+			(type default)
+		)
+	)
+	(wire
+		(pts
 			(xy 135.89 100.33) (xy 146.05 100.33)
 		)
@@
 	)
 	(symbol
-		(lib_id "power:GND")
-		(at 64.77 124.46 0)
-		(unit 1)
-		(exclude_from_sim no)
-		(in_bom yes)
-		(on_board yes)
-		(dnp no)
-		(fields_autoplaced yes)
-		(property "Reference" "#PWR011"
-			(at 64.77 130.81 0)
-			(effects
-				(font
-					(size 1.27 1.27)
-				)
-				(hide yes)
-			)
-		)
-		(property "Value" "GND"
-			(at 64.77 128.5955 0)
-			(effects
-				(font
-					(size 1.27 1.27)
-				)
-			)
-		)
-		(property "Footprint" ""
-			(at 64.77 124.46 0)
-			(effects
-				(font
-					(size 1.27 1.27)
-				)
-				(hide yes)
-			)
-		)
-		(property "Datasheet" ""
-			(at 64.77 124.46 0)
-			(effects
-				(font
-					(size 1.27 1.27)
-				)
-				(hide yes)
-			)
-		)
-		(property "Description" ""
-			(at 64.77 124.46 0)
-			(effects
-				(font
-					(size 1.27 1.27)
-				)
-				(hide yes)
-			)
-		)
-		(pin "1"
-		)
-		(instances
-			(project "motherboard"
-				(path "/4cf1c087-5c32-4958-ab30-5e92afc4ef4b/8d1ce991-8a62-4e08-8a5e-b7da93c506d5"
-					(reference "#PWR011")
-					(unit 1)
-				)
-			)
-		)
-	)
-	(symbol
 		(lib_id "Device:R")
 		(at 55.88 72.39 180)
@@
 	(symbol
 		(lib_id "Device:R")
-		(at 64.77 119.38 180)
+		(at 63.5 72.39 180)
 		(unit 1)
 		(exclude_from_sim no)
@@
 		(dnp no)
 		(property "Reference" "R6"
-			(at 63.754 124.714 90)
+			(at 62.484 77.724 90)
 			(effects
 				(font
@@
 		)
 		(property "Value" "10k"
-			(at 65.024 121.158 90)
+			(at 63.754 74.168 90)
 			(effects
 				(font
@@
 		)
 		(property "Footprint" "Resistor_THT:R_Axial_DIN0204_L3.6mm_D1.6mm_P7.62mm_Horizontal"
-			(at 66.548 119.38 90)
+			(at 65.278 72.39 90)
 			(effects
 				(font
@@
 		)
 		(property "Datasheet" "~"
-			(at 64.77 119.38 0)
+			(at 63.5 72.39 0)
 			(effects
 				(font
@@
 		)
 		(property "Description" "Resistor"
-			(at 64.77 119.38 0)
+			(at 63.5 72.39 0)
 			(effects
 				(font
