File: prototypes/motherboard-stage2_take3/power.kicad_sch (KiCad schematic)
At the start: 14 parts, among them J3 Power, J4 PowerLed, J5 Reset, U10 BA05CCOT, U11 MAX708, U9 74HCT373

Commit message: Finalized stage 2
Other:
- moved on the sheet: C36
Changed lines of the file:
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@@
 	(wire
 		(pts
-			(xy 48.26 147.32) (xy 48.26 149.86)
-		)
-		(stroke
-			(width 0)
-			(type default)
-		)
-	)
-	(wire
-		(pts
-			(xy 48.26 135.89) (xy 48.26 139.7)
+			(xy 264.16 73.66) (xy 264.16 76.2)
+		)
+		(stroke
+			(width 0)
+			(type default)
+		)
+	)
+	(wire
+		(pts
+			(xy 264.16 62.23) (xy 264.16 66.04)
 		)
 		(stroke
@@
 	(wire
 		(pts
-			(xy 247.65 31.75) (xy 248.92 31.75)
+			(xy 247.65 31.75) (xy 261.62 31.75)
 		)
 		(stroke
@@
 		(pts
 			(xy 99.06 81.28) (xy 97.79 81.28)
+		)
+		(stroke
+			(width 0)
+			(type default)
+		)
+	)
+	(wire
+		(pts
+			(xy 261.62 31.75) (xy 261.62 34.29)
 		)
 		(stroke
@@
 	(hierarchical_label "~{RST}"
 		(shape output)
-		(at 248.92 31.75 0)
+		(at 261.62 34.29 270)
 		(fields_autoplaced yes)
 		(effects
@@
 				(size 1.27 1.27)
 			)
-			(justify left)
+			(justify right)
 		)
 	)
@@
 	(symbol
 		(lib_id "power:GND")
-		(at 48.26 149.86 0)
+		(at 264.16 76.2 0)
 		(unit 1)
 		(exclude_from_sim no)
@@
 		(fields_autoplaced yes)
 		(property "Reference" "#PWR091"
-			(at 48.26 156.21 0)
+			(at 264.16 82.55 0)
 			(effects
 				(font
@@
 		)
 		(property "Value" "GND"
-			(at 48.26 153.9955 0)
+			(at 264.16 80.3355 0)
 			(effects
 				(font
@@
 		)
 		(property "Footprint" ""
-			(at 48.26 149.86 0)
+			(at 264.16 76.2 0)
 			(effects
 				(font
@@
 		)
 		(property "Datasheet" ""
-			(at 48.26 149.86 0)
+			(at 264.16 76.2 0)
 			(effects
 				(font
@@
 		)
 		(property "Description" ""
-			(at 48.26 149.86 0)
+			(at 264.16 76.2 0)
 			(effects
 				(font
@@
 	(symbol
 		(lib_id "power:VCC")
-		(at 48.26 135.89 0)
+		(at 264.16 62.23 0)
 		(unit 1)
 		(exclude_from_sim no)
@@
 		(fields_autoplaced yes)
 		(property "Reference" "#PWR090"
-			(at 48.26 139.7 0)
+			(at 264.16 66.04 0)
 			(effects
 				(font
@@
 		)
 		(property "Value" "VCC"
-			(at 48.26 132.3881 0)
+			(at 264.16 58.7281 0)
 			(effects
 				(font
@@
 		)
 		(property "Footprint" ""
-			(at 48.26 135.89 0)
+			(at 264.16 62.23 0)
 			(effects
 				(font
@@
 		)
 		(property "Datasheet" ""
-			(at 48.26 135.89 0)
+			(at 264.16 62.23 0)
 			(effects
 				(font
@@
 		)
 		(property "Description" ""
-			(at 48.26 135.89 0)
+			(at 264.16 62.23 0)
 			(effects
 				(font
@@
 	(symbol
 		(lib_id "Device:C")
-		(at 48.26 143.51 0)
+		(at 264.16 69.85 0)
 		(unit 1)
 		(exclude_from_sim no)
@@
 		(fields_autoplaced yes)
 		(property "Reference" "C36"
-			(at 51.181 142.8663 0)
+			(at 267.081 69.2063 0)
 			(effects
 				(font
@@
 		)
 		(property "Value" "100n"
-			(at 51.181 144.7873 0)
+			(at 267.081 71.1273 0)
 			(effects
 				(font
@@
 		)
 		(property "Footprint" "Capacitor_THT:C_Disc_D5.0mm_W2.5mm_P2.50mm"
-			(at 49.2252 147.32 0)
+			(at 265.1252 73.66 0)
 			(effects
 				(font
@@
 		)
 		(property "Datasheet" "~"
-			(at 48.26 143.51 0)
+			(at 264.16 69.85 0)
 			(effects
 				(font
@@
 		)
 		(property "Description" ""
-			(at 48.26 143.51 0)
-			(effects
-				(font
+			(at 264.16 69.85 0)
+			(effects
+				(font
