File: prototypes/motherboard-stage2_take3/serial.kicad_sch (KiCad schematic)
At the start: 20 parts, among them J7 POT Con, J8 Console, J9 DE9_Plug, U12 65c22, U13 XR88C92, U14 MAX232, U15 MCP2221A, Y2 3.3864

Commit message: Finalized stage 2
Parts:
- added JP1: Reset EN, Connector_PinHeader_2.54mm:PinHeader_1x02_P2.54mm_Vertical, symbol Jumper:Jumper_2_Open
Connections:
- net ~{RST}: now also JP1.2 (B); no longer U15.4 (~{RST})
- new net: JP1.1 (A), U15.4 (~{RST})
Other:
- moved on the sheet: C15, C16, C19, C20, C21, C22, C23, J8, J9, U13, U14, U15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
