File: motherboard/motherboard-stage2/irq_handler.kicad_sch (KiCad schematic)
At the start: 16 parts, among them U16 74HCT02, U17 74HCT148, U18 74HCT148, U19 74HCT574, U20 74HCT00, U21 74HCT574, U22 74HCT85

Commit message: Ordered stage 2!
Connections:
- net VCC: no longer U16.11, U16.12
- net ~{IRQ}: now also U16.13; no longer U22.7 (Oa<b)
- net at U21.4 (D2), U22.14 (B2): now also U20.6; no longer U20.11
- net at U21.2 (D0), U22.9 (B0): now also U20.11; no longer U20.6
- net at U16.10: now also U21.1 (OE); no longer U21.11 (Cp)
- net at U16.1, U16.8, U16.9: no longer U21.1 (OE)
- new net: U16.11, U16.12, U22.7 (Oa<b)
- new net Q: U21.11 (Cp)
- no-connect marks 15 -> 14
Other:
- moved on the sheet: U16C, U16D, U22
