File: motherboard/motherboard-stage2/motherboard.kicad_sch (KiCad schematic)
At the start: 6 parts

Commit message: Ordered stage 2!
Other:
- sheet IRQ-Handler ports: added Q; removed none
Changed lines of the file:
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@@
+	)
+	(junction
+		(at 88.9 135.89)
+		(diameter 0)
+		(color 0 0 0 0)
 	)
 	(junction
@@
 	(wire
 		(pts
-			(xy 45.72 135.89) (xy 176.53 135.89)
+			(xy 45.72 135.89) (xy 88.9 135.89)
 		)
 		(stroke
@@
 	(wire
 		(pts
+			(xy 88.9 82.55) (xy 88.9 135.89)
+		)
+		(stroke
+			(width 0)
+			(type default)
+		)
+	)
+	(wire
+		(pts
 			(xy 161.29 110.49) (xy 182.88 110.49)
 		)
@@
 		(pts
 			(xy 68.58 156.21) (xy 68.58 142.24)
+		)
+		(stroke
+			(width 0)
+			(type default)
+		)
+	)
+	(wire
+		(pts
+			(xy 88.9 135.89) (xy 176.53 135.89)
 		)
 		(stroke
@@
 	)
 	(label "AM[14..21]"
-		(at 83.82 130.81 0)
+		(at 115.57 130.81 0)
 		(fields_autoplaced yes)
 		(effects
@@
 	)
 	(label "~{IRQ_[0..15]}"
-		(at 83.82 121.92 0)
+		(at 115.57 121.92 0)
 		(fields_autoplaced yes)
 		(effects
@@
 	)
 	(label "A[0..15]"
-		(at 86.36 128.27 0)
+		(at 115.57 128.27 0)
 		(fields_autoplaced yes)
 		(effects
@@
 			(effects
 				(font
+					(size 1.27 1.27)
+				)
+				(justify left)
+			)
+		)
+		(pin "Q" input
+			(at 88.9 82.55 270)
+			(effects
+				(font
