File: pototypes/usb-adapter/usb-adapter.kicad_pcb (KiCad board)
At the start: 6 copper layers, 10.5 x 19 mm, 6 parts, among them J1 Conn_02x07_Counter_Clockwise, U2 CP2102N-Axx-xQFN20, U3 TXB0104RGY, U4 AP130-33Y

Commit message: Updates to a lot!
Parts:
- removed U4: AP130-33Y, Package_TO_SOT_SMD:SOT-89-3
- added R3: 22k1, PCM_Resistor_SMD_AKL:R_0402_1005Metric_Pad0.72x0.64mm, F.Cu at (98.0, 87.2)
- added R4: 47k5, PCM_Resistor_SMD_AKL:R_0402_1005Metric_Pad0.72x0.64mm, F.Cu at (95.5, 87.2)
- added U1: USBLC6-2SC6, Package_TO_SOT_SMD:SOT-23-6, F.Cu at (96.8, 77.5)
- moved U3 2.46 mm to (96.8, 82.8)
- moved R1 0.81 mm to (98.0, 88.4)
- moved R2 0.81 mm to (95.5, 88.4)
- moved U2 0.31 mm to (96.7, 92.4)
Connections:
- J1 pad 1: +5V -> unconnected-(J1-Pin_1-Pad1)
- J1 pad 11: unconnected-(J1-Pin_11-Pad11) -> +5V
- R1 pad 1: +3.3V -> RST
- R1 pad 2: RST -> Net-(J1-Pin_4)
- R2 pad 1: RST -> GND
- U2 pad 4: USB-DP -> Net-(U2-D+)
- U2 pad 5: USB-DM -> Net-(U2-D-)
- U2 pad 7: unconnected-(U2-VREGIN-Pad7) -> +5V
- U2 pad 8: unconnected-(U2-VBUS-Pad8) -> Net-(U2-VBUS)
Routing:
- net RST: track 12.1 -> 0.00 mm
- net USB-DP: track 18.4 -> 6.48 mm, vias 1 -> 0
- net Net-(J1-Pin_6): track 10.4 -> 0.00 mm, vias 1 -> 0
- net USB-DM: track 16.2 -> 6.42 mm, vias 1 -> 0
- net Net-(J1-Pin_5): track 9.29 -> 0.00 mm, vias 1 -> 0
- net +5V: track 10.6 -> 1.59 mm, vias 1 -> 4
- net +3.3V: track 10.0 -> 1.74 mm, vias 4 -> 3
- net Net-(J1-Pin_3): track 7.55 -> 0.00 mm, vias 2 -> 0
- net TX: track 5.98 -> 0.00 mm, vias 2 -> 0
- net CTS: track 5.66 -> 0.00 mm, vias 2 -> 0
- net RX: track 5.44 -> 0.00 mm, vias 2 -> 0
- net RTS: track 5.07 -> 0.00 mm, vias 2 -> 0
- net Net-(J1-Pin_4): track 4.29 -> 0.00 mm
- net GND: track 8.02 -> 5.99 mm, vias 8 -> 1
- net Net-(U2-VBUS): track 0.00 -> 1.22 mm
- added copper zone on In2.Cu, net GND
Other:
- board size 10.5 x 19 mm -> 10.5 x 20.7 mm
- board text added: "3.3v"
- board text added: "5v"
- board text added: "GND"
