File: motherboard/WIP/motherboard-stage3-take2/irq_handler.kicad_sch (KiCad schematic)
At the start: 16 parts, among them U16 74HCT02, U17 74HCT148, U18 74HCT148, U19 74HCT574, U20 74HCT00, U21 74HCT574, U22 74HCT85

Commit message: Ordered stage 2!
Connections:
- net at U16.10: now also U21.1 (OE); no longer U21.11 (Cp)
- net at U16.1, U16.8, U16.9: no longer U21.1 (OE)
- new net Q: U21.11 (Cp)
Changed lines of the file:
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@@
-	)
-	(junction
-		(at 87.63 139.7)
-		(diameter 0)
-		(color 0 0 0 0)
 	)
 	(junction
@@
 	(wire
 		(pts
+			(xy 116.84 132.08) (xy 104.14 132.08)
+		)
+		(stroke
+			(width 0)
+			(type default)
+		)
+	)
+	(wire
+		(pts
 			(xy 120.65 156.21) (xy 120.65 127)
 		)
@@
 		)
 	)
-	(wire
-		(pts
-			(xy 104.14 132.08) (xy 123.19 132.08)
-		)
-		(stroke
-			(width 0)
-			(type default)
-		)
-	)
 	(bus
 		(pts
@@
 	(wire
 		(pts
-			(xy 123.19 132.08) (xy 123.19 78.74)
-		)
-		(stroke
-			(width 0)
-			(type default)
-		)
-	)
-	(wire
-		(pts
 			(xy 153.67 73.66) (xy 157.48 73.66)
 		)
@@
 	(wire
 		(pts
-			(xy 116.84 81.28) (xy 116.84 139.7)
+			(xy 116.84 81.28) (xy 116.84 132.08)
 		)
 		(stroke
@@
 	(wire
 		(pts
-			(xy 87.63 139.7) (xy 116.84 139.7)
+			(xy 127 78.74) (xy 128.27 78.74)
 		)
 		(stroke
@@
 		(pts
 			(xy 46.99 102.87) (xy 60.96 102.87)
-		)
-		(stroke
-			(width 0)
-			(type default)
-		)
-	)
-	(wire
-		(pts
-			(xy 123.19 78.74) (xy 128.27 78.74)
 		)
 		(stroke
@@
 		(fields_autoplaced yes)
 		(effects
+			(font
+				(size 1.27 1.27)
+			)
+			(justify right)
+		)
+	)
+	(hierarchical_label "Q"
+		(shape input)
+		(at 127 78.74 180)
+		(fields_autoplaced yes)
+		(effects

Commit message: Updated stage 2 and stage 3, and started on a cf addon
Other:
- title: IRQ Handler -> MicroLind - IRQ Handler
Changed lines of the file:
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@@
 	(paper "A4")
 	(title_block
-		(title "IRQ Handler")
-		(date "2024-02-03")
-		(rev "1")
+		(title "MicroLind - IRQ Handler")
+		(date "2025-03-03")
+		(rev "C0")
 		(company "Eric Lind")
 	)

Commit message: Updates to a lot!
Connections:
- net GND: no longer U22.2 (Ia<b), U22.3 (Ia=b), U22.4 (Ia>b)
- net VCC: now also U22.2 (Ia<b), U22.3 (Ia=b), U22.4 (Ia>b); no longer U16.11, U16.12
- net ~{IRQ}: now also U16.13; no longer U22.7 (Oa<b)
- new net: U16.11, U16.12, U22.7 (Oa<b)
Other:
- moved on the sheet: U16D
Changed lines of the file:
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@@
 	)
 	(junction
-		(at 261.62 36.83)
-		(diameter 0)
-		(color 0 0 0 0)
-	)
-	(junction
 		(at 45.72 165.1)
 		(diameter 0)
@@
 	)
 	(junction
-		(at 156.21 114.3)
-		(diameter 0)
-		(color 0 0 0 0)
-	)
-	(junction
 		(at 222.25 144.78)
 		(diameter 0)
@@
 	)
 	(junction
+		(at 156.21 127)
+		(diameter 0)
+		(color 0 0 0 0)
+	)
+	(junction
+		(at 156.21 109.22)
+		(diameter 0)
+		(color 0 0 0 0)
+	)
+	(junction
 		(at 156.21 111.76)
 		(diameter 0)
@@
 	(wire
 		(pts
-			(xy 261.62 36.83) (xy 264.16 36.83)
-		)
-		(stroke
-			(width 0)
-			(type default)
-		)
-	)
-	(wire
-		(pts
 			(xy 153.67 109.22) (xy 156.21 109.22)
 		)
@@
 	(wire
 		(pts
-			(xy 261.62 36.83) (xy 261.62 41.91)
+			(xy 113.03 58.42) (xy 113.03 87.63)
 		)
 		(stroke
@@
 	(wire
 		(pts
-			(xy 113.03 58.42) (xy 113.03 87.63)
+			(xy 241.3 45.72) (xy 241.3 46.99)
 		)
 		(stroke
@@
 	(wire
 		(pts
-			(xy 241.3 45.72) (xy 241.3 46.99)
+			(xy 156.21 127) (xy 156.21 129.54)
 		)
 		(stroke
@@
 	(wire
 		(pts
-			(xy 153.67 127) (xy 158.75 127)
+			(xy 153.67 127) (xy 156.21 127)
 		)
 		(stroke
@@
 	(wire
 		(pts
-			(xy 156.21 114.3) (xy 156.21 138.43)
-		)
-		(stroke
-			(width 0)
-			(type default)
-		)
-	)
-	(wire
-		(pts
 			(xy 198.12 144.78) (xy 198.12 146.05)
 		)
@@
 	(wire
 		(pts
-			(xy 261.62 41.91) (xy 264.16 41.91)
-		)
-		(stroke
-			(width 0)
-			(type default)
-		)
-	)
-	(wire
-		(pts
 			(xy 120.65 127) (xy 128.27 127)
 		)
@@
 	(wire
 		(pts
+			(xy 156.21 127) (xy 156.21 124.46)
+		)
+		(stroke
+			(width 0)
+			(type default)
+		)
+	)
+	(wire
+		(pts
 			(xy 46.99 162.56) (xy 45.72 162.56)
 		)
@@
 		)
 	)
+	(wire
+		(pts
+			(xy 156.21 100.33) (xy 156.21 109.22)
+		)
+		(stroke
+			(width 0)
+			(type default)
+		)
+	)
 	(bus
 		(pts
@@
 	(wire
 		(pts
-			(xy 261.62 31.75) (xy 261.62 36.83)
-		)
-		(stroke
-			(width 0)
-			(type default)
-		)
-	)
-	(wire
-		(pts
 			(xy 222.25 154.94) (xy 222.25 153.67)
 		)
@@
 	(wire
 		(pts
+			(xy 171.45 127) (xy 173.99 127)
+		)
+		(stroke
+			(width 0)
+			(type default)
+		)
+	)
+	(wire
+		(pts
 			(xy 87.63 71.12) (xy 87.63 54.61)
 		)
@@
 	(hierarchical_label "~{IRQ}"
 		(shape output)
-		(at 158.75 127 0)
+		(at 173.99 127 0)
 		(fields_autoplaced yes)
 		(effects
@@
 	)
 	(symbol
-		(lib_id "power:VCC")
-		(at 261.62 31.75 0)
-		(mirror y)
-		(unit 1)
-		(exclude_from_sim no)
-		(in_bom yes)
-		(on_board yes)
-		(dnp no)
-		(fields_autoplaced yes)
-		(property "Reference" "#PWR067"
-			(at 261.62 35.56 0)
-			(effects
-				(font
-					(size 1.27 1.27)
-				)
-				(hide yes)
-			)
-		)
-		(property "Value" "VCC"
-			(at 261.62 28.2481 0)
-			(effects
-				(font
-					(size 1.27 1.27)
-				)
-			)
-		)
-		(property "Footprint" ""
-			(at 261.62 31.75 0)
-			(effects
-				(font
-					(size 1.27 1.27)
-				)
-				(hide yes)
-			)
-		)
-		(property "Datasheet" ""
-			(at 261.62 31.75 0)
-			(effects
-				(font
-					(size 1.27 1.27)
-				)
-				(hide yes)
-			)
-		)
-		(property "Description" ""
-			(at 261.62 31.75 0)
-			(effects
-				(font
-					(size 1.27 1.27)
-				)
-				(hide yes)
-			)
-		)
-		(pin "1"
-		)
-		(instances
-			(project "motherboard"
-				(path "/4cf1c087-5c32-4958-ab30-5e92afc4ef4b/8bee193f-f974-40fd-8292-ec5c594bf5d7"
-					(reference "#PWR067")
-					(unit 1)
-				)
-			)
-		)
-	)
-	(symbol
 		(lib_id "74xx:74LS00")
 		(at 102.87 87.63 0)
@@
 	)
 	(symbol
+		(lib_id "power:VCC")
+		(at 156.21 100.33 0)
+		(mirror y)
+		(unit 1)
+		(exclude_from_sim no)
+		(in_bom yes)
+		(on_board yes)
+		(dnp no)
+		(fields_autoplaced yes)
+		(property "Reference" "#PWR060"
+			(at 156.21 104.14 0)
+			(effects
+				(font
+					(size 1.27 1.27)
+				)
+				(hide yes)
+			)
+		)
+		(property "Value" "VCC"
+			(at 156.21 96.8281 0)
+			(effects
+				(font
+					(size 1.27 1.27)
+				)
+			)
+		)
+		(property "Footprint" ""
+			(at 156.21 100.33 0)
+			(effects
+				(font
+					(size 1.27 1.27)
+				)
+				(hide yes)
+			)
+		)
+		(property "Datasheet" ""
+			(at 156.21 100.33 0)
+			(effects
+				(font
+					(size 1.27 1.27)
+				)
+				(hide yes)
+			)
+		)
+		(property "Description" ""
+			(at 156.21 100.33 0)
+			(effects
+				(font
+					(size 1.27 1.27)
+				)
+				(hide yes)
+			)
+		)
+		(pin "1"
+		)
+		(instances
+			(project "motherboard"
+				(path "/4cf1c087-5c32-4958-ab30-5e92afc4ef4b/8bee193f-f974-40fd-8292-ec5c594bf5d7"
+					(reference "#PWR060")
+					(unit 1)
+				)
+			)
+		)
+	)
+	(symbol
 		(lib_id "Device:C")
 		(at 233.68 149.86 0)
@@
 	)
 	(symbol
-		(lib_id "power:GND")
-		(at 156.21 138.43 0)
-		(mirror y)
-		(unit 1)
-		(exclude_from_sim no)
-		(in_bom yes)
-		(on_board yes)
-		(dnp no)
-		(fields_autoplaced yes)
-		(property "Reference" "#PWR060"
-			(at 156.21 144.78 0)
-			(effects
-				(font
-					(size 1.27 1.27)
-				)
-				(hide yes)
-			)
-		)
-		(property "Value" "GND"
-			(at 156.21 142.5655 0)
-			(effects
-				(font
-					(size 1.27 1.27)
-				)
-			)
-		)
-		(property "Footprint" ""
-			(at 156.21 138.43 0)
-			(effects
-				(font
-					(size 1.27 1.27)
-				)
-				(hide yes)
-			)
-		)
-		(property "Datasheet" ""
-			(at 156.21 138.43 0)
-			(effects
-				(font
-					(size 1.27 1.27)
-				)
-				(hide yes)
-			)
-		)
-		(property "Description" ""
-			(at 156.21 138.43 0)
-			(effects
-				(font
-					(size 1.27 1.27)
-				)
-				(hide yes)
-			)
-		)
-		(pin "1"
-		)
-		(instances
-			(project "motherboard"
-				(path "/4cf1c087-5c32-4958-ab30-5e92afc4ef4b/8bee193f-f974-40fd-8292-ec5c594bf5d7"
-					(reference "#PWR060")
-					(unit 1)
-				)
-			)
-		)
-	)
-	(symbol
 		(lib_id "power:VCC")
 		(at 73.66 40.64 0)
@@
 	(symbol
 		(lib_id "74xx:74HCT02")
-		(at 271.78 39.37 0)
+		(at 163.83 127 0)
 		(unit 4)
 		(exclude_from_sim no)
@@
 		(fields_autoplaced yes)
 		(property "Reference" "U16"
-			(at 271.78 32.5501 0)
+			(at 163.83 120.1801 0)
 			(effects
 				(font
@@
 		)
 		(property "Value" "74HCT02"
-			(at 271.78 34.4711 0)
+			(at 163.83 122.1011 0)
 			(effects
 				(font
@@
 		)
 		(property "Footprint" "Package_DIP:DIP-14_W7.62mm_Socket"
-			(at 271.78 39.37 0)
+			(at 163.83 127 0)
 			(effects
 				(font
@@
 		)
 		(property "Datasheet" "http://www.ti.com/lit/gpn/sn74hct02"
-			(at 271.78 39.37 0)
+			(at 163.83 127 0)
 			(effects
 				(font
@@
 		)
 		(property "Description" ""
-			(at 271.78 39.37 0)
+			(at 163.83 127 0)
 			(effects
 				(font

Commit message: Updates
Changed lines of the file:
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@@
 (kicad_sch
-	(version 20231120)
+	(version 20250114)
 	(generator "eeschema")
-	(generator_version "8.0")
+	(generator_version "9.0")
 	(paper "A4")
 	(title_block
@@
 	(label "~{IRQ_9}"
 		(at 34.29 62.23 0)
-		(fields_autoplaced yes)
 		(effects
 			(font
@@
 	(label "~{IRQ_4}"
 		(at 34.29 105.41 0)
-		(fields_autoplaced yes)
 		(effects
 			(font
@@
 	(label "~{IRQ_6}"
 		(at 48.26 100.33 0)
-		(fields_autoplaced yes)
 		(effects
 			(font
@@
 	(label "D1"
 		(at 153.67 58.42 0)
-		(fields_autoplaced yes)
 		(effects
 			(font
@@
 	(label "~{IRQ_2}"
 		(at 34.29 113.03 0)
-		(fields_autoplaced yes)
 		(effects
 			(font
@@
 	(label "D7"
 		(at 81.28 161.29 0)
-		(fields_autoplaced yes)
 		(effects
 			(font
@@
 	(label "D7"
 		(at 153.67 73.66 0)
-		(fields_autoplaced yes)
 		(effects
 			(font
@@
 	(label "~{IRQ_5}"
 		(at 34.29 102.87 0)
-		(fields_autoplaced yes)
 		(effects
 			(font
@@
 	(label "D4"
 		(at 153.67 66.04 0)
-		(fields_autoplaced yes)
 		(effects
 			(font
@@
 	(label "~{IRQ_14}"
 		(at 48.26 52.07 0)
-		(fields_autoplaced yes)
 		(effects
 			(font
@@
 	(label "~{IRQ_3}"
 		(at 48.26 107.95 0)
-		(fields_autoplaced yes)
 		(effects
 			(font
@@
 	(label "~{IRQ_13}"
 		(at 48.26 54.61 0)
-		(fields_autoplaced yes)
 		(effects
 			(font
@@
 	(label "D6"
 		(at 81.28 158.75 0)
-		(fields_autoplaced yes)
 		(effects
 			(font
@@
 	(label "D[0..7]"
 		(at 162.56 46.99 0)
-		(fields_autoplaced yes)
 		(effects
 			(font
@@
 	(label "~{IRQ_4}"
 		(at 48.26 105.41 0)
-		(fields_autoplaced yes)
 		(effects
 			(font
@@
 	(label "D5"
 		(at 81.28 156.21 0)
-		(fields_autoplaced yes)
 		(effects
 			(font
@@
 	(label "~{IRQ_9}"
 		(at 48.26 64.77 0)
-		(fields_autoplaced yes)
 		(effects
 			(font
@@
 	(label "~{IRQ_10}"
 		(at 48.26 62.23 0)
-		(fields_autoplaced yes)
 		(effects
 			(font
@@
 	(label "~{IRQ_7}"
 		(at 48.26 97.79 0)
-		(fields_autoplaced yes)
 		(effects
 			(font
@@
 	(label "D6"
 		(at 153.67 71.12 0)
-		(fields_autoplaced yes)
 		(effects
 			(font
@@
 	(label "~{IRQ_12}"
 		(at 34.29 57.15 0)
-		(fields_autoplaced yes)
 		(effects
 			(font
@@
 	(label "~{IRQ_5}"
 		(at 48.26 102.87 0)
-		(fields_autoplaced yes)
 		(effects
 			(font
@@
 	(label "~{IRQ_7}"
 		(at 34.29 97.79 0)
-		(fields_autoplaced yes)
 		(effects
 			(font
@@
 	(label "~{IRQ_11}"
 		(at 48.26 59.69 0)
-		(fields_autoplaced yes)
 		(effects
 			(font
@@
 	(label "~{IRQ_13}"
 		(at 34.29 54.61 0)
-		(fields_autoplaced yes)
 		(effects
 			(font
@@
 	(label "~{IRQ_11}"
 		(at 34.29 67.31 0)
-		(fields_autoplaced yes)
 		(effects
 			(font
@@
 	(label "~{IRQ_8}"
 		(at 34.29 59.69 0)
-		(fields_autoplaced yes)
 		(effects
 			(font
@@
 	(label "~{IRQ_1}"
 		(at 48.26 113.03 0)
-		(fields_autoplaced yes)
 		(effects
 			(font
@@
 	(label "~{IRQ_1}"
 		(at 34.29 110.49 0)
-		(fields_autoplaced yes)
 		(effects
 			(font
@@
 	(label "~{IRQ_[0..15]}"
 		(at 35.56 39.37 0)
-		(fields_autoplaced yes)
 		(effects
 			(font
@@
 	(label "~{IRQ_0}"
 		(at 48.26 115.57 0)
-		(fields_autoplaced yes)
 		(effects
 			(font
@@
 	(label "D[0..7]"
 		(at 74.93 149.86 0)
-		(fields_autoplaced yes)
 		(effects
 			(font
@@
 	(label "D2"
 		(at 153.67 60.96 0)
-		(fields_autoplaced yes)
 		(effects
 			(font
@@
 	(label "D5"
 		(at 153.67 68.58 0)
-		(fields_autoplaced yes)
 		(effects
 			(font
@@
 	(label "~{IRQ_12}"
 		(at 48.26 57.15 0)
-		(fields_autoplaced yes)
 		(effects
 			(font
@@
 	(label "D0"
 		(at 153.67 55.88 0)
-		(fields_autoplaced yes)
 		(effects
 			(font
@@
 	(label "~{IRQ_8}"
 		(at 48.26 67.31 0)
-		(fields_autoplaced yes)
 		(effects
 			(font
@@
 	(label "~{IRQ_2}"
 		(at 48.26 110.49 0)
-		(fields_autoplaced yes)
 		(effects
 			(font
@@
 	(label "~{IRQ_0}"
 		(at 34.29 107.95 0)
-		(fields_autoplaced yes)
 		(effects
 			(font
@@
 	(label "~{IRQ_14}"
 		(at 34.29 52.07 0)
-		(fields_autoplaced yes)
 		(effects
 			(font
@@
 	(label "~{IRQ_3}"
 		(at 34.29 115.57 0)
-		(fields_autoplaced yes)
 		(effects
 			(font
@@
 	(label "~{IRQ_6}"
 		(at 34.29 100.33 0)
-		(fields_autoplaced yes)
 		(effects
 			(font
@@
 	(label "D3"
 		(at 153.67 63.5 0)
-		(fields_autoplaced yes)
 		(effects
 			(font
@@
 	(label "~{IRQ_10}"
 		(at 34.29 64.77 0)
-		(fields_autoplaced yes)
 		(effects
 			(font
@@
 	(label "D4"
 		(at 81.28 153.67 0)
-		(fields_autoplaced yes)
 		(effects
 			(font
@@
 		(shape output)
 		(at 173.99 127 0)
-		(fields_autoplaced yes)
 		(effects
 			(font
@@
 		(shape input)
 		(at 44.45 173.99 180)
-		(fields_autoplaced yes)
 		(effects
 			(font
@@
 		(shape input)
 		(at 127 78.74 180)
-		(fields_autoplaced yes)
 		(effects
 			(font
@@
 		(shape input)
 		(at 34.29 39.37 180)
-		(fields_autoplaced yes)
 		(effects
 			(font
@@
 		(shape input)
 		(at 73.66 149.86 180)
-		(fields_autoplaced yes)
 		(effects
 			(font
@@
 		(shape input)
 		(at 44.45 165.1 180)
-		(fields_autoplaced yes)
 		(effects
 			(font
@@
 		(shape input)
 		(at 44.45 157.48 180)
-		(fields_autoplaced yes)
 		(effects
 			(font
@@
 		(shape input)
 		(at 170.18 46.99 0)
-		(fields_autoplaced yes)
 		(effects
 			(font
