File: peripherals/WIP/VideoExpansionCard-VDC8568/videoexpansioncard-vdc.kicad_pcb (KiCad board)
At the start: 2 copper layers, 94 x 147.6 mm, 30 parts, among them J1 VEP, J2 DE9_Plug, Q1 2SC1815, U1 8568, U4 74HCT244, U5 74LS07, U6 74HCT273, U7 GAL16V8, U8 27C64, X1 ACO-16MHz

Commit message: Updates to a lot!
Parts:
- moved X1 102.2 mm to (127.9, 77.7)
- moved U7 83.7 mm to (38.4, 68.2)
- moved U6 81.5 mm to (15.9, 103.9)
- moved U8 54.4 mm to (32.9, 96.6)
- moved U2 52.8 mm to (94.0, 124.5)
- moved C4 43.4 mm to (15.6, 99.1)
- moved C5 42.3 mm to (56.7, 81.3)
- moved U1 40.5 mm to (71.1, 86.4)
- moved U3 17.6 mm to (94.0, 91.4)
- moved J1 0.36 mm to (55.9, 160.0)

Commit message: A lot of updates
Parts:
- removed U6: 74HCT273, Package_DIP:DIP-20_W7.62mm_Socket
- removed U7: GAL16V8, Package_DIP:DIP-20_W7.62mm_Socket
- removed U8: 27C64, Package_DIP:DIP-28_W15.24mm
- moved C1 39.4 mm to (44.5, 73.5), turned to 90 degrees
- moved X1 27.7 mm to (100.3, 80.0)
- moved C4 22.0 mm to (19.1, 77.3), turned to 90 degrees
- moved U1 11.4 mm to (66.0, 76.2)
- moved FB7 3.81 mm to (99.1, 48.2)
- moved FB6 3.17 mm to (95.2, 48.1)
- moved FB5 2.54 mm to (91.4, 48.2)
- moved FB4 1.91 mm to (87.6, 48.2)
- moved FB3 1.27 mm to (83.8, 48.2)
- moved FB2 0.63 mm to (80.0, 48.1)
Connections:
- net V_SYNC renamed Net-(U1-VSYNC)
- J1 pad 5: unconnected-(J1-Pin_5-Pad5) -> E
- U1 pad 5: VCD_CS -> E
- U1 pad 9: ~{VDC_CHIP_IRQ} -> ~{RST}
