File: peripherals/WIP/VideoExpansionCard-VDC8568/videoexpansioncard-vdc.kicad_pcb (KiCad board)
At the start: 2 copper layers, 94 x 147.6 mm, 27 parts, among them J1 VEP, J2 DE9_Plug, Q1 2SC1815, U1 8568, U4 74HCT244, U5 74LS07, X1 ACO-16MHz

Commit message: Latest state of HW
Parts:
- added C6: 220nF, Capacitor_THT:C_Disc_D5.0mm_W2.5mm_P2.50mm, F.Cu at (26.7, 30.5)
- added C7: 220nF, Capacitor_THT:C_Disc_D5.0mm_W2.5mm_P2.50mm, F.Cu at (20.3, 30.5)
- added J3: LP, Connector_PinHeader_2.54mm:PinHeader_1x01_P2.54mm_Vertical, F.Cu at (36.9, 108.5)
- added JP1: Interupt Source, Connector_PinHeader_2.54mm:PinHeader_1x03_P2.54mm_Vertical, F.Cu at (36.9, 98.8)
- added U9: 74HCT00, Package_DIP:DIP-14_W7.62mm_Socket, F.Cu at (24.9, 98.6)
- C1, C4: footprint Capacitor_THT:C_Axial_L3.8mm_D2.6mm_P7.50mm_Horizontal -> Capacitor_THT:C_Disc_D5.0mm_W2.5mm_P2.50mm
- C2, C3: value 220nF -> 100nF; footprint Capacitor_THT:C_Axial_L3.8mm_D2.6mm_P7.50mm_Horizontal -> Capacitor_THT:C_Disc_D5.0mm_W2.5mm_P2.50mm
- C5: footprint Capacitor_THT:CP_Radial_D4.0mm_P1.50mm -> Capacitor_THT:CP_Radial_D5.0mm_P2.00mm
- moved C1 54.3 mm to (90.2, 102.9), turned to -90 degrees
- moved C5 36.5 mm to (85.9, 103.2), turned to -90 degrees
- moved C4 25.8 mm to (28.7, 53.5), turned to -90 degrees
- moved U4 14.7 mm to (61.0, 67.4), turned to 90 degrees
- moved U5 10.7 mm to (32.5, 61.5), turned to 90 degrees
- moved U2 8.48 mm to (95.2, 116.1)
- moved U3 1.38 mm to (95.3, 92.0)
Connections:
- net Net-(U1-VSYNC) renamed HSYNC
- U1 pad 25: unconnected-(U1-LPEN-Pad25) -> Net-(J3-Pin_1)
- U1 pad 9: ~{RST} -> ~{INT}
