File: peripherals/WIP/ExpansionBoard/ExpansionBoard.kicad_pcb (KiCad board)
At the start: 4 copper layers, 170.2 x 170.2 mm, 46 parts, among them J1 ExpansionPort_IN, J10 ExpansionPort_OUT, J11 I2C Header, J12 Ext. I2C, J2 Exp 1A, J3 Exp 1B, J4 Exp 2A, J5 Exp 2B, J6 Exp 3, J7 Exp 4, J8 Exp 5, J9 Exp 6, Q1 BC337, SW1 SW_DIP_x04, U1 8259A, U2 AS6C4008-55PCN, U27 GAL 22V10, U3 AS6C4008-55PCN, U4 Motherboard Outline, U5 GAL16V8, U6 74LS245, U7 74LS540

Commit message: Latest state of HW
Parts:
- removed U5: GAL16V8, Package_DIP:DIP-20_W7.62mm_Socket
- added U8: 74AHCT138, Package_DIP:DIP-16_W7.62mm_Socket, F.Cu at (147.3, 179.0)
- moved G*** 88.8 mm to (80.1, 124.5)
- moved C1 2.54 mm to (34.9, 156.3)
- moved C2 2.54 mm to (34.9, 181.6)
- moved J11 2.54 mm to (86.4, 196.8)
- moved U2 2.54 mm to (38.1, 171.4)
- moved U3 2.54 mm to (38.1, 196.8)
- moved C13 0.67 mm to (119.4, 69.8)
- moved C15 0.67 mm to (94.0, 69.8)
- moved C11 0.54 mm to (144.8, 69.8)
- moved C17 0.54 mm to (68.6, 69.8)
- moved C19 0.54 mm to (43.2, 69.8)
- moved C9 0.54 mm to (170.2, 69.8)
- moved J10 0.13 mm to (29.0, 93.0)
- moved J5 0.13 mm to (152.4, 80.0)
Connections:
- net /~{EXP_EN} renamed ~{EXP_EN}
- net BOARD_SEL renamed /auto-config/BOARD_ADDRESS_SELECT
- net ~{IRQ_EN} renamed /AddressDecoder/~{IRQ_EN}
- J1 pad 2: /~{RST} -> ~{RST}
- J1 pad 29: /~{RAMX_EN} -> ~{RAMX_EN}
- J1 pad 3: /~{BREQ} -> ~{BREQ}
- J1 pad 4: /~{EXP_IRQ_L} -> ~{EXP_IRQ_L}
- J1 pad 41: /~{MAP_EN} -> ~{MAP_EN}
- J1 pad 42: /A14 -> A14
- J1 pad 44: /A15 -> A15
- J1 pad 45: /AM20 -> AM20
- J1 pad 46: /AM21 -> AM21
- J1 pad 5: /E -> E
- J1 pad 6: /R/~{W} -> R/~{W}
- J1 pad 7: /BAVAIL -> BAVAIL
- J1 pad 9: /AM19 -> AM19
- J10 pad 2: /~{RST} -> ~{RST}
- J10 pad 29: /~{RAMX_EN} -> ~{RAMX_EN}
- J10 pad 3: /~{BREQ} -> ~{BREQ}
- J10 pad 4: /~{EXP_IRQ_R} -> ~{EXP_IRQ_R}
- J10 pad 41: /~{MAP_EN} -> ~{MAP_EN}
- J10 pad 42: /A14 -> A14
- J10 pad 44: /A15 -> A15
- J10 pad 45: /AM20 -> AM20
- J10 pad 46: /AM21 -> AM21
- J10 pad 5: /E -> E
- J10 pad 6: /R/~{W} -> R/~{W}
- J10 pad 7: /BAVAIL -> BAVAIL
- J10 pad 9: /AM19 -> AM19
- JP1 pad 1: /InteruptController/~{EXP_IRQ_L} -> ~{EXP_IRQ_L}
- JP1 pad 3: /InteruptController/~{EXP_IRQ_R} -> ~{EXP_IRQ_R}
- JP2 pad 1: /InteruptController/~{EXP_IRQ_L} -> ~{EXP_IRQ_L}
- JP2 pad 3: /InteruptController/~{EXP_IRQ_R} -> ~{EXP_IRQ_R}
- RN1 pad 5: ~{I2C_DETECT} -> /auto-config/~{I2C_DETECT}
- RN1 pad 6: ~{RTC_DETECT} -> /auto-config/~{RTC_DETECT}
- U27 pad 11: unconnected-(U27-I11-Pad11) -> ~{RAMX_EN}
- U27 pad 14: ~{SLOT6_EN} -> Net-(U27-I010)
- U27 pad 15: ~{SLOT5_EN} -> Net-(U27-IO9)
- U27 pad 16: ~{SLOT4_EN} -> Net-(U27-IO8)
- U27 pad 17: ~{SLOT3_EN} -> AM21
- U27 pad 18: ~{SLOT2_EN} -> AM20
- U27 pad 19: ~{SLOT1_EN} -> AM19
- U27 pad 20: unconnected-(U27-IO4-Pad20) -> ~{RAMX_H_EN}
- U27 pad 21: ~{I2C_EN} -> ~{RAMX_L_EN}
- U27 pad 23: unconnected-(U27-IO1-Pad23) -> /AddressDecoder/~{INFO_EN}
- U6 pad 15: ~{RTC_DETECT} -> /auto-config/~{RTC_DETECT}
- U6 pad 16: ~{I2C_DETECT} -> /auto-config/~{I2C_DETECT}
- U6 pad 19: ~{INFO_EN} -> /AddressDecoder/~{INFO_EN}
Routing:
- net A0: track 0.00 -> 521.6 mm, vias 0 -> 5
- net ~{RD}: track 0.00 -> 518.7 mm, vias 0 -> 5
- net A1: track 0.00 -> 497.5 mm, vias 0 -> 5
- net ~{WR}: track 0.00 -> 490.3 mm, vias 0 -> 4
- net D0: track 0.00 -> 477.3 mm, vias 0 -> 4
- net A2: track 0.00 -> 477.3 mm, vias 0 -> 4
- net D1: track 0.00 -> 471.5 mm, vias 0 -> 4
- net D2: track 0.00 -> 465.1 mm, vias 0 -> 4
- net D7: track 0.00 -> 449.6 mm, vias 0 -> 4
- net D6: track 0.00 -> 447.7 mm, vias 0 -> 4
- net D5: track 0.00 -> 445.3 mm, vias 0 -> 4
- net D4: track 0.00 -> 444.3 mm, vias 0 -> 4
- net D3: track 0.00 -> 442.9 mm, vias 0 -> 3
- net A3: track 0.00 -> 374.4 mm, vias 0 -> 4
- net A4: track 0.00 -> 330.2 mm, vias 0 -> 3
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- added copper zone on In1.Cu, net VCC
