File: peripherals/WIP/ExpansionBoard/InteruptController.kicad_sch (KiCad schematic)
At the start: 0 parts

Commit message: Updates
Parts:
- added C2, C5: 100n, Capacitor_THT:C_Disc_D3.0mm_W1.6mm_P2.50mm, symbol Device:C
- added U1: 8259A, Package_DIP:DIP-28_W15.24mm_Socket, symbol Interface:8259A
- added U7: 74LS540, Package_DIP:DIP-20_W7.62mm_Socket, symbol 74xx:74LS540
Connections:
- new net: U1.18 (IR0), U7.11 (Y7)
- new net: U1.19 (IR1), U7.12 (Y6)
- new net: U1.20 (IR2), U7.13 (Y5)
- new net: U1.21 (IR3), U7.14 (Y4)
- new net: U1.22 (IR4), U7.15 (Y3)
- new net: U1.23 (IR5), U7.16 (Y2)
- new net: U1.24 (IR6), U7.17 (Y1)
- new net A0: U1.27 (A0)
- new net D0: U1.11 (D0)
- new net D1: U1.10 (D1)
- new net D2: U1.9 (D2)
- new net D3: U1.8 (D3)
- new net D4: U1.7 (D4)
- new net D5: U1.6 (D5)
- new net D6: U1.5 (D6)
- new net D7: U1.4 (D7)
- new net EXP_IRQ: U1.17 (INT), U7.2 (A0)
- new net GND: C2.2, C5.2, U1.14 (GND), U1.25 (IR7), U7.1 (G1), U7.10 (GND), U7.19 (G2)
- new net VCC: C2.1, C5.1, U1.16 (~{SP}/~{EN}), U1.26 (~{INTA}), U1.28 (VCC), U7.20 (VCC)
- new net ~{EX_IRQ}: U7.18 (Y0)
- new net ~{I2C_IRQ}: U7.3 (A1)
- new net ~{IRQ_E1}: U7.9 (A7)
- new net ~{IRQ_E2}: U7.8 (A6)
- new net ~{IRQ_E3}: U7.7 (A5)
- new net ~{IRQ_E4}: U7.6 (A4)
- new net ~{IRQ_E5}: U7.5 (A3)
- new net ~{IRQ_E6}: U7.4 (A2)
- new net ~{IRQ_EN}: U1.1 (~{CS})
- new net ~{RD}: U1.3 (~{RD})
- new net ~{WR}: U1.2 (~{WR})
- no-connect marks 0 -> 3

Commit message: Updatesto Expansion
Parts:
- added JP1, JP2: Jumper_3_Open, Connector_PinHeader_2.54mm:PinHeader_1x03_P2.54mm_Vertical, symbol Jumper:Jumper_3_Open
- added Q1: BC337, Package_TO_SOT_THT:TO-92, symbol Simulation_SPICE:NPN
- added R1: 4k7, Resistor_THT:R_Axial_DIN0207_L6.3mm_D2.5mm_P7.62mm_Horizontal, symbol Device:R
Connections:
- net GND: now also Q1.3 (E); no longer U1.25 (IR7)
- net EXP_IRQ: no longer names the net of U7.2 (A0)
- net EXP_IRQ: now also JP1.2 (C); no longer U1.17 (INT)
- net ~{EX_IRQ}: no longer names the net of U7.18 (Y0)
- net ~{EX_IRQ}: now also U1.25 (IR7)
- new net: JP2.2 (C), Q1.1 (C)
- new net: Q1.2 (B), R1.1
- new net: R1.2, U1.17 (INT)
- new net ~{EXP_IRQ_L}: JP1.1 (A), JP2.1 (A)
- new net ~{EXP_IRQ_R}: JP1.3 (B), JP2.3 (B)
Other:
- note added: "IRQ7 function is not final!"
