File: peripherals/WIP/ExpansionBoard/auto-config.kicad_sch (KiCad schematic)
At the start: 7 parts, among them U5 TCA9548APWR, U7 MCP7940N-xP, Y1 32.768kHz

Commit message: Updates
Parts:
- removed BT1: Battery_Cell, symbol Device:Battery_Cell
- removed R1, R2: 4k7, symbol Device:R
- removed U5: TCA9548APWR, Package_SO:TSSOP-24_4.4x7.8mm_P0.65mm, symbol Interface_Expansion:TCA9548APWR
- removed U7: MCP7940N-xP, symbol Timer_RTC:MCP7940N-xP
- removed U9: ~, symbol New_Library:PCA9564
- removed Y1: 32.768kHz, symbol Device:Crystal_Small
- added C1: 100n, Capacitor_THT:C_Disc_D3.0mm_W1.6mm_P2.50mm, symbol Device:C
- added RN1: 10k, Resistor_THT:R_Array_SIP7, symbol Device:R_Network06
- added SW1: SW_DIP_x04, Connector_PinHeader_2.54mm:PinHeader_2x04_P2.54mm_Vertical, symbol Switch:SW_DIP_x04
- added U6: 74LS245, Package_DIP:DIP-20_W7.62mm_Socket, symbol 74xx:74LS245
Connections:
- net GND: now also C1.2, SW1.5, SW1.6, SW1.7, SW1.8, U6.1 (A->B), U6.10 (GND), U6.11 (B7)
- net VCC: now also C1.1, RN1.1 (common), U6.20 (VCC)
- new net BOARD_SEL: SW1.3
- new net D0: U6.2 (A0)
- new net D1: U6.3 (A1)
- new net D2: U6.4 (A2)
- new net D3: U6.5 (A3)
- new net D4: U6.6 (A4)
- new net D5: U6.7 (A5)
- new net D6: U6.8 (A6)
- new net D7: U6.9 (A7)
- new net MEM1_EN: RN1.2 (R1), SW1.1, U6.18 (B0)
- new net MEM2_EN: RN1.3 (R2), SW1.2, U6.17 (B1)
- new net SPARE: RN1.4 (R3), SW1.4, U6.14 (B4)
- new net ~{I2C_DETECT}: RN1.5 (R4), U6.16 (B2)
- new net ~{INFO_EN}: U6.19 (CE)
- new net ~{RTC_DETECT}: RN1.6 (R5), U6.15 (B3)
- no-connect marks 0 -> 3
