File: motherboard/WIP/motherboard-stage3-Rev1/ps2.kicad_sch (KiCad schematic)
At the start: 15 parts, among them J17 PS2_DEBUG_TX, U9 ATmega88, Y3 32.768kHz

Commit message: Removed PS2 from next gen microlind, due to unsolved hardware issues
Parts:
- P9: value ~ -> (none)
