File: motherboard/motherboard-stage3/irq_handler.kicad_sch (KiCad schematic)
At the start: 16 parts, among them U16 74HCT02, U17 74HCT148, U18 74HCT148, U19 74HCT574, U20 74HCT00, U21 74HCT574, U22 74HCT85

Commit message: Latest state of HW
Connections:
- net GND: now also U19.6 (D4), U19.7 (D5), U19.8 (D6), U19.9 (D7)
- net VCC: now also U17.10 (IO)
- no-connect marks 15 -> 10
Changed lines of the file:
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@@
 	)
 	(junction
+		(at 86.36 168.91)
+		(diameter 0)
+		(color 0 0 0 0)
+	)
+	(junction
 		(at 209.55 144.78)
 		(diameter 0)
@@
 	)
 	(junction
+		(at 86.36 171.45)
+		(diameter 0)
+		(color 0 0 0 0)
+	)
+	(junction
 		(at 198.12 144.78)
 		(diameter 0)
@@
 	)
 	(junction
+		(at 86.36 166.37)
+		(diameter 0)
+		(color 0 0 0 0)
+	)
+	(junction
+		(at 86.36 179.07)
+		(diameter 0)
+		(color 0 0 0 0)
+	)
+	(junction
 		(at 156.21 127)
 		(diameter 0)
@@
 	)
 	(no_connect
-		(at 87.63 163.83)
-	)
-	(no_connect
 		(at 153.67 124.46)
 	)
@@
 	)
 	(no_connect
-		(at 87.63 168.91)
-	)
-	(no_connect
 		(at 86.36 64.77)
 	)
@@
 	)
 	(no_connect
-		(at 60.96 49.53)
-	)
-	(no_connect
-		(at 87.63 166.37)
-	)
-	(no_connect
 		(at 86.36 62.23)
 	)
@@
 		(at 113.03 168.91)
 	)
-	(no_connect
-		(at 87.63 171.45)
-	)
 	(bus_entry
 		(at 160.02 53.34)
@@
 	(wire
 		(pts
+			(xy 86.36 171.45) (xy 86.36 179.07)
+		)
+		(stroke
+			(width 0)
+			(type default)
+		)
+	)
+	(wire
+		(pts
 			(xy 113.03 156.21) (xy 120.65 156.21)
 		)
@@
 	(wire
 		(pts
+			(xy 87.63 163.83) (xy 86.36 163.83)
+		)
+		(stroke
+			(width 0)
+			(type default)
+		)
+	)
+	(wire
+		(pts
 			(xy 73.66 40.64) (xy 73.66 41.91)
 		)
@@
 		)
 	)
+	(wire
+		(pts
+			(xy 86.36 168.91) (xy 86.36 171.45)
+		)
+		(stroke
+			(width 0)
+			(type default)
+		)
+	)
 	(bus
 		(pts
@@
 	(wire
 		(pts
+			(xy 86.36 166.37) (xy 87.63 166.37)
+		)
+		(stroke
+			(width 0)
+			(type default)
+		)
+	)
+	(wire
+		(pts
 			(xy 209.55 144.78) (xy 222.25 144.78)
 		)
@@
 	(wire
 		(pts
+			(xy 86.36 168.91) (xy 87.63 168.91)
+		)
+		(stroke
+			(width 0)
+			(type default)
+		)
+	)
+	(wire
+		(pts
 			(xy 113.03 87.63) (xy 113.03 114.3)
 		)
@@
 	(wire
 		(pts
+			(xy 86.36 171.45) (xy 87.63 171.45)
+		)
+		(stroke
+			(width 0)
+			(type default)
+		)
+	)
+	(wire
+		(pts
 			(xy 115.57 109.22) (xy 115.57 115.57)
 		)
@@
 	(wire
 		(pts
+			(xy 86.36 166.37) (xy 86.36 168.91)
+		)
+		(stroke
+			(width 0)
+			(type default)
+		)
+	)
+	(wire
+		(pts
 			(xy 33.02 97.79) (xy 41.91 97.79)
 		)
@@
 	(wire
 		(pts
+			(xy 58.42 49.53) (xy 58.42 45.72)
+		)
+		(stroke
+			(width 0)
+			(type default)
+		)
+	)
+	(wire
+		(pts
 			(xy 256.54 144.78) (xy 267.97 144.78)
 		)
@@
 	(wire
 		(pts
+			(xy 86.36 163.83) (xy 86.36 166.37)
+		)
+		(stroke
+			(width 0)
+			(type default)
+		)
+	)
+	(wire
+		(pts
 			(xy 19.05 49.53) (xy 22.86 49.53)
 		)
@@
 	(wire
 		(pts
+			(xy 58.42 49.53) (xy 60.96 49.53)
+		)
+		(stroke
+			(width 0)
+			(type default)
+		)
+	)
+	(wire
+		(pts
 			(xy 73.66 125.73) (xy 73.66 127)
 		)
@@
 					(unit 1)
 				)
+			)
+		)
+	)
+	(symbol
+		(lib_id "power:VCC")
+		(at 58.42 45.72 0)
+		(mirror y)
+		(unit 1)
+		(body_style 1)
+		(exclude_from_sim no)
+		(in_bom yes)
+		(on_board yes)
+		(in_pos_files yes)
+		(dnp no)
+		(fields_autoplaced yes)
+		(property "Reference" "#PWR096"
+			(at 58.42 49.53 0)
+			(hide yes)
+			(show_name no)
+			(do_not_autoplace no)
+			(effects
+				(font
+					(size 1.27 1.27)
+				)
+			)
+		)
+		(property "Value" "VCC"
+			(at 58.42 42.2181 0)
+			(show_name no)
+			(do_not_autoplace no)
+			(effects
+				(font
+					(size 1.27 1.27)
+				)
+			)
+		)
+		(property "Footprint" ""
+			(at 58.42 45.72 0)
+			(hide yes)
+			(show_name no)
+			(do_not_autoplace no)
+			(effects
+				(font
+					(size 1.27 1.27)
+				)
+			)
+		)
+		(property "Datasheet" ""
+			(at 58.42 45.72 0)
+			(hide yes)
+			(show_name no)
+			(do_not_autoplace no)
+			(effects
+				(font
+					(size 1.27 1.27)
+				)
+			)
+		)
+		(property "Description" ""
+			(at 58.42 45.72 0)
+			(hide yes)
+			(show_name no)
+			(do_not_autoplace no)
+			(effects
+				(font
+					(size 1.27 1.27)
+				)
+			)
+		)
+		(pin "1"
+		)
+		(instances
+			(project "motherboard"
+				(path "/4cf1c087-5c32-4958-ab30-5e92afc4ef4b/8bee193f-f974-40fd-8292-ec5c594bf5d7"
+					(reference "#PWR096")
+					(unit 1)
+				)
