File: motherboard/motherboard-stage3/serial.kicad_sch (KiCad schematic)
At the start: 35 parts, among them J10 CTS, J11 RTS, J12 MEM, J13 EX1, J14 EX2, J15 FUT, J3 Reset EN, J4 PowerLed, J6 PC Speaker, J7 POT Con, J8 Clock Exp., J9 LPen, P5 Console, P6 Serial, P8 Joystic Ports, U12 65c22, U13 XR88C92, U14 MAX232, U15 MCP2221A, Y2 3.3864

Commit message: Latest state of HW
Parts:
- added C36: 1u, Capacitor_THT:CP_Radial_D4.0mm_P2.00mm, symbol Device:C_Polarized
Connections:
- net GND: now also C21.1, U13.40 (IP2), U13.5 (IP1), U14.10 (T2IN), U14.8 (R2IN), C36.2
- net VCC: no longer C22.1, U15.1 (VDD)
- net at C23.1, P5.1 (VBUS): now also U15.1 (VDD); no longer U15.11 (VUSB)
- net at U14.2 (VS+): now also C36.1; no longer C21.1
- new net: C22.1, U15.11 (VUSB)
- no-connect marks 25 -> 21
Other:
- moved on the sheet: P6
